Commit message: Inverse Kinematics applied IKSrv created which gives res to apply_ik client

File: ws/simulation_ws/src/aspha18_urdf/urdf/aspha18.urdf (robot description, URDF)
Before this commit: robot aspha18_urdf, 18 links, 17 joints
Joints:
- joint base_rotation: limit effort=0 velocity=0 -> effort=0 velocity=0.3
- joint gripper_joint: limit lower=-1.2 upper=1.9 effort=0 velocity=0 -> lower=-1.2 upper=1.9 effort=0.1 velocity=0.1
- joint wheel_rotate2: axis 1 0 0 -> -1 0 0
- joint wheel_rotate4: axis 1 0 0 -> -1 0 0
