Commit message: Inverse kinematics added with gripper camera

File: ws/rover_ws/src/isac/urdf/robot_2link.urdf (robot description, URDF)
Before this commit: robot flat, 6 links, 5 joints
Joints:
- joint elbow_joint: limit lower=-3.14 upper=3.14 effort=0 velocity=0.1 -> effort=0 velocity=0.3
- joint gripper_joint: limit lower=-1.2 upper=1.9 effort=0 velocity=0.1 -> effort=0 velocity=0.3
- joint shoulder_joint: limit lower=-0.45 upper=1.12 effort=0 velocity=0.1 -> effort=0 velocity=0.3

File: ws/simulation_ws/src/aspha18_urdf/urdf/aspha18.urdf (robot description, URDF)
Before this commit: robot aspha18_urdf, 18 links, 17 joints
Links:
- added link camera_link_arm, mass 1e-5; collision box size=0.05 0.05 0.05; visual box size=0.05 0.05 0.05
Joints:
- added joint camera_joint_arm: type fixed, parent gripper, child camera_link_arm, origin xyz=0.0 0.13 -0.2 rpy=0 1.57 1.57, axis 0 0 0
- joint base_rotation: limit effort=0 velocity=0.3 -> lower=-3.14 upper=3.14 effort=0 velocity=0.3
- joint elbow_joint: limit lower=-3.14 upper=3.14 effort=0 velocity=0.1 -> lower=-3.14 upper=3.14 effort=0 velocity=0.3
- joint gripper_joint: limit lower=-1.2 upper=1.9 effort=0.1 velocity=0.1 -> lower=-3.14 upper=3.14 effort=0 velocity=0.3
- joint shoulder_joint: limit lower=-0.45 upper=1.12 effort=0 velocity=0.1 -> lower=-3.14 upper=3.14 effort=0 velocity=0.3
